Commit message: feat: add Rebot vertical peg-in-hole task

File: peg_insert_reproduction/rebot_assets/rebot_description/urdf/rebot.urdf (robot description, URDF)
Before this commit: robot robot, 11 links, 10 joints
Links:
- removed link gripper_motor_link
Joints:
- removed joint Joint_7
- joint Joint_1: limit lower=-1.57079633 upper=1.57079633 effort=100 velocity=3.0 -> lower=-1.570796326794897 upper=1.570796326794897 effort=20 velocity=3
- joint Joint_2: limit lower=3.14159265 upper=4.71238898 effort=100 velocity=3.0 -> lower=0.0 upper=3.1415926 effort=20 velocity=3
- joint Joint_3: limit lower=2.92203023 upper=5.27822472 effort=100 velocity=3.0 -> lower=-3.141592653589793 upper=0.0 effort=20 velocity=3
- joint Joint_4: limit lower=-1.35123391 upper=1.79035875 effort=100 velocity=3.0 -> lower=-1.570796326794897 upper=1.570796326794897 effort=20 velocity=3
- joint Joint_5: limit lower=-3.14159265 upper=0.00000000 effort=100 velocity=3.0 -> lower=-1.570796326794897 upper=1.570796326794897 effort=20 velocity=3
- joint Joint_6: limit lower=-4.71238898 upper=1.57079633 effort=100 velocity=3.0 -> lower=-1.570796326794897 upper=1.570796326794897 effort=20 velocity=3
- joint Joint_ee_1: axis 0 0 1 -> 0 0 -1; limit lower=0 upper=0.08 effort=100 velocity=0.1 -> lower=0 upper=0.05 effort=100 velocity=0.1
- joint Joint_ee_2: axis 0 0 1 -> 0 0 -1; limit lower=0 upper=0.08 effort=100 velocity=0.1 -> lower=0 upper=0.05 effort=100 velocity=0.1; mimic (none) -> joint=Joint_ee_1 multiplier=1 offset=0
