Commit message: feat: sync Rebot Isaac model to XML baseline, add joint friction DR
- Align bridge URDF/runtime cfg with rebot.xml (J2 0-180 deg, 3 rad/s, effort 50)
- Randomize arm joint Coulomb/viscous friction on reset
- Add velocity-limit and XML-hash checks to verify_rebot_model_sync.py
- Add pre-training smoke test script
- Rewrite HANDOFF for the retraining and sim-to-sim workflow

Co-Authored-By: Claude Code <noreply@anthropic.com>

File: peg_insert_reproduction/rebot_assets/rebot_description/urdf/rebot.urdf (robot description, URDF)
Before this commit: robot robot, 10 links, 9 joints
Joints:
- joint Joint_1: limit lower=-1.570796326794897 upper=1.570796326794897 effort=20 velocity=3 -> lower=-1.570796326794897 upper=1.570796326794897 effort=50 velocity=3
- joint Joint_2: limit lower=0.0 upper=3.1415926 effort=20 velocity=3 -> lower=0.0 upper=3.141592653589793 effort=50 velocity=3
- joint Joint_3: limit lower=-3.141592653589793 upper=0.0 effort=20 velocity=3 -> lower=-3.141592653589793 upper=0.0 effort=50 velocity=3
- joint Joint_4: limit lower=-1.570796326794897 upper=1.570796326794897 effort=20 velocity=3 -> lower=-1.570796326794897 upper=1.570796326794897 effort=50 velocity=3
- joint Joint_5: limit lower=-1.570796326794897 upper=1.570796326794897 effort=20 velocity=3 -> lower=-1.570796326794897 upper=1.570796326794897 effort=50 velocity=3
- joint Joint_6: limit lower=-1.570796326794897 upper=1.570796326794897 effort=20 velocity=3 -> lower=-1.570796326794897 upper=1.570796326794897 effort=50 velocity=3
